File: projects/dollar_tinyml/hardware/dml20m/dml20m.kicad_sch (KiCad schematic)
At the start: 36 parts, among them J1 USB_A, J2 Conn_ARM_SWD_TagConnect_TC203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, J3 Header 2.54mm, J4 Header 2.54mm, Q1 BC547B, SW1 SW_Push, U1 LIS2DH12, U2 LP4054HB5F, U3 PY32F003F18U6TR, U4 XC6206PxxxMR, U5 BM7161

Commit message: dollarml: dml20m revision ready for production
Parts:
- BT1: value Battery_Cell -> LIR1225; now not fitted
- BZ1: now left out of the parts list
- D1: value LED_RGB -> LED 5050-6P-GRB; MPN (none) -> TC5050RGBF08-3CJH-AF53A; Manufacturer (none) -> TCWIN
- J3, J4: now not fitted; now left out of the parts list
- R11: value 100R -> 120R
- SW1: value SW_Push -> PTS647SM50SMTR2LFS; MPN (none) -> PTS647SM50SMTR2LFS; Manufacturer (none) -> C&K
- U1: MPN (none) -> LIS2DH12TR; Manufacturer (none) -> ST Microelectronics
- U2: value LP4054HB5F -> Li charger 4054; LCSC C517187 -> (none); MPN (none) -> LP4054HB5F; Manufacturer (none) -> LOWPOWER
- U3: LCSC C3018713 -> (none); MPN (none) -> PY32F003F18U6TR; Manufacturer (none) -> PUYA)
- U4: value XC6206PxxxMR -> XC6206P332MR; MPN (none) -> XC6206P332MR; Manufacturer (none) -> Torex
- U5: now not fitted
Other:
- note removed: "FIXME: verify microcontroller and accelerometer pinout"
- note removed: "FIXME: verify transistor and buzzer pinout"
Changed lines of the file:
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@@
 		)
 	)
-	(text "FIXME: verify transistor and buzzer pinout"
-		(exclude_from_sim no)
-		(at 233.934 151.384 0)
-		(effects
-			(font
-				(size 1.27 1.27)
-			)
-		)
-	)
 	(text "Microcontroller"
 		(exclude_from_sim no)
@@
 	(text "LiIon/LiPo battery\n3.7V nominal, 4.2v max"
 		(exclude_from_sim no)
-		(at 92.71 27.305 0)
+		(at 55.372 59.944 0)
+		(effects
+			(font
+				(size 1.27 1.27)
+			)
+			(justify left bottom)
+		)
+	)
+	(text "LiIon/LiPo battery\n3.7V nominal, 4.2v max"
+		(exclude_from_sim no)
+		(at 96.52 33.274 0)
 		(effects
 			(font
@@
 		)
 	)
-	(text "FIXME: verify microcontroller and accelerometer pinout\n"
-		(exclude_from_sim no)
-		(at 57.404 117.094 0)
-		(effects
-			(font
-				(size 1.27 1.27)
-			)
-		)
-	)
 	(text "Headers"
 		(exclude_from_sim no)
@@
 			)
 		)
-		(property "Value" "100R"
+		(property "Value" "120R"
 			(at 249.809 144.526 90)
 			(effects
@@
 			)
 		)
-		(property "Value" "XC6206PxxxMR"
+		(property "Value" "XC6206P332MR"
 			(at 133.35 34.29 0)
 			(effects
@@
 			)
 		)
+		(property "MPN" "XC6206P332MR"
+			(at 133.35 38.1 0)
+			(effects
+				(font
+					(size 1.27 1.27)
+				)
+				(hide yes)
+			)
+		)
+		(property "Manufacturer" "Torex"
+			(at 133.35 38.1 0)
+			(effects
+				(font
+					(size 1.27 1.27)
+				)
+				(hide yes)
+			)
+		)
 		(pin "3"
 		)
@@
 		(unit 1)
 		(exclude_from_sim no)
-		(in_bom yes)
+		(in_bom no)
 		(on_board yes)
-		(dnp no)
+		(dnp yes)
 		(property "Reference" "J3"
 			(at 135.636 138.176 0)
@@
 			)
 		)
+		(property "Manufacturer" "ST Microelectronics"
+			(at 50.8 166.37 0)
+			(effects
+				(font
+					(size 1.27 1.27)
+				)
+				(hide yes)
+			)
+		)
+		(property "MPN" "LIS2DH12TR"
+			(at 50.8 166.37 0)
+			(effects
+				(font
+					(size 1.27 1.27)
+				)
+				(hide yes)
+			)
+		)
 		(pin "6"
 		)
@@
 		(unit 1)
 		(exclude_from_sim no)
-		(in_bom yes)
+		(in_bom no)
 		(on_board yes)
 		(dnp no)
@@
 			)
 		)
-		(property "Value" "LP4054HB5F"
+		(property "Value" "Li charger 4054"
 			(at 73.025 29.21 0)
 			(effects
@@
 			)
 		)
-		(property "LCSC" "C517187"
+		(property "Manufacturer" "LOWPOWER"
+			(at 83.82 38.1 0)
+			(effects
+				(font
+					(size 1.27 1.27)
+				)
+				(hide yes)
+			)
+		)
+		(property "MPN" "LP4054HB5F"
 			(at 83.82 38.1 0)
 			(effects
@@
 			)
 		)
-		(property "Value" "LED_RGB"
+		(property "Value" "LED 5050-6P-GRB"
 			(at 240.03 81.28 0)
 			(effects
@@
 			)
 		)
+		(property "Manufacturer" "TCWIN"
+			(at 240.03 92.71 0)
+			(effects
+				(font
+					(size 1.27 1.27)
+				)
+				(hide yes)
+			)
+		)
+		(property "MPN" "TC5050RGBF08-3CJH-AF53A"
+			(at 240.03 92.71 0)
+			(effects
+				(font
+					(size 1.27 1.27)
+				)
+				(hide yes)
+			)
+		)
 		(pin "6"
 		)
@@
 			)
 		)
-		(property "Value" "SW_Push"
+		(property "Value" "PTS647SM50SMTR2LFS"
 			(at 204.47 138.4299 90)
 			(effects
@@
 			)
 		)
+		(property "Manufacturer" " C&K"
+			(at 203.2 137.16 90)
+			(effects
+				(font
+					(size 1.27 1.27)
+				)
+				(hide yes)
+			)
+		)
+		(property "MPN" "PTS647SM50SMTR2LFS"
+			(at 203.2 137.16 90)
+			(effects
+				(font
+					(size 1.27 1.27)
+				)
+				(hide yes)
+			)
+		)
 		(pin "2"
 		)
@@
 		(in_bom no)
 		(on_board yes)
-		(dnp no)
+		(dnp yes)
 		(fields_autoplaced yes)
 		(property "Reference" "U5"
@@
 		(unit 1)
 		(exclude_from_sim no)
-		(in_bom yes)
+		(in_bom no)
 		(on_board yes)
-		(dnp no)
+		(dnp yes)
 		(property "Reference" "J4"
 			(at 135.636 158.496 0)
@@
 			)
 		)
-		(property "Datasheet" "https://datasheet.lcsc.com/lcsc/2302231730_WCH-Jiangsu-Qin-Heng-CH32V003F4U6_C5299908.pdf"
+		(property "Datasheet" ""
 			(at 116.84 74.93 0)
 			(effects
@@
 			)
 		)
-		(property "LCSC" "C3018713"
+		(property "Manufacturer" "PUYA)"
+			(at 116.84 107.95 0)
+			(effects
+				(font
+					(size 1.27 1.27)
+				)
+				(hide yes)
+			)
+		)
+		(property "MPN" "PY32F003F18U6TR"
 			(at 116.84 107.95 0)
 			(effects
@@
 		(in_bom no)
 		(on_board yes)
-		(dnp no)
+		(dnp yes)
 		(fields_autoplaced yes)
 		(property "Reference" "BT1"
@@
 			)
 		)
-		(property "Value" "Battery_Cell"
+		(property "Value" "LIR1225"
 			(at 113.03 44.5135 0)
 			(effects
