File: projects/dollar_tinyml/hardware/dml21m/dml21m.kicad_sch (KiCad schematic)
At the start: 32 parts, among them J2 Conn_ARM_SWD_TagConnect_TC203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, J4 Header 2.54mm, J5 USB_C_Receptacle_PowerOnly_6P, Q1 BC547B, SW1 PTS647SM50SMTR2LFS, U1 LIS2DH12, U2 Li charger 4054, U3 PY32F003F18U6TR, U4 XC6206P332MR

Commit message: dollarml: More sketches on next board
Parts:
- added U5: PUYA P25Q16SH-SSH-IT, Package_SO:SOIC-8_5.3x5.3mm_P1.27mm, symbol Memory_Flash:W25Q32JVSS
- added U6: BM7161, dml10:BM7161, symbol dml10:BM7161
Connections:
- net BLE_INT: now also U6.1 (IRQ)
- net BLE_SCL: now also U6.2 (SCL)
- net BLE_SDA: now also U6.3 (SDA)
- net GND: now also U5.4 (GND), U6.5 (GND)
- net VDD: now also U5.8 (VCC), U6.4 (VDD)
- net LED_BLUE_P: no longer names the net of U3.5 (PA12)
- net LED_RED_P: no longer names the net of U3.3 (PA7)
Other:
- note added: "BC7161 is non-standard I2C, and should be alone on bus"
- note added: "Bluetooth"
- note added: "FIXME: check pinout, wire Share with SWD?"
- note added: "FIXME: switch to CH32V006F8U6"
- note added: "Holtek BLE beacon"
- moved on the sheet: SW1
